File: rev_c/mbino.sch (KiCad schematic (older format))
At the start: 52 parts, among them J1 HEADER_1X3, SW1 KSS221GLFS, U1 L78M05CDT-TR, U2 MCP1700T-3302E-SOT89, U3 MCP2551_SOIC8, U4 ATMEGA324_QFP44, X1 16MHz

Commit message: Added MakerBus reset circuit.
Parts:
- added C13, C14: .1uF, symbol C
- added R10: 180, symbol R_HORIZ
- added R11: 10K, symbol R_VERT
- added U5: 74x2G06, symbol 74XV2G06
- U1: value L78M05CDT-TR -> L78L05CDT-TR
- renumbered C2 to C1, C1 to C2
Connections:
- net labels added: 3V3, 5V, VCC
- wire segments 200 -> 212
Other:
- moved on the sheet: C10, C2, C4, C5, C6, C7, C8, C9, H1, H2, H3, H4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
